File: Hardware/Bottom/Winston-BOTTOM.sch (EAGLE design)
At the start: 31 parts, among them U1 AD5242-SO16

Commit message: updated top and bottom boards with everything from Take 002
Parts:
- added J1: (no value), LinnesLab-Connectors:CONN_07
Connections:
- removed net LED.CTRL: U$4.A
- removed net PPG: C21.2, OP3G$1.OUT, U1.B2
- removed net TIA: C10.2, C15.1, OP4G$1.OUT, U1.W1
- new net A0/PPG: C21.2, J1.5, OP3G$1.OUT, U1.B2
- new net A7/TIA: C10.2, C15.1, J1.6, OP4G$1.OUT, U1.W1
- new net D29/LED.CTRL: J1.4, U$4.A
- new net N$11: J1.1
- new net N$6: J1.3
- new net N$7: J1.2
Changed lines of the file:
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@@
 <part name="GND30" library="LinnesLab-Symbols" deviceset="GND" device=""/>
 <part name="SUPPLY24" library="LinnesLab-Symbols" deviceset="3.3V" device=""/>
+<part name="J1" library="LinnesLab-Connectors" deviceset="CONN_07" device=""/>
 </parts>
 <sheets>
@@
 <attribute name="VALUE" x="17.78" y="-7.366" size="1.778" layer="96" align="bottom-center"/>
 </instance>
+<instance part="J1" gate="G$1" x="104.14" y="-25.4" smashed="yes">
+<attribute name="VALUE" x="99.06" y="-35.306" size="1.778" layer="96" font="vector"/>
+<attribute name="NAME" x="99.06" y="-12.192" size="1.778" layer="95" font="vector"/>
+</instance>
 </instances>
 <busses>
@@
 </segment>
 </net>
-<net name="TIA" class="0">
+<net name="A7/TIA" class="0">
 <segment>
 <wire x1="132.08" y1="30.48" x2="127" y2="30.48" width="0.1524" layer="91"/>
@@
 <junction x="83.82" y="111.76"/>
 </segment>
+<segment>
+<pinref part="J1" gate="G$1" pin="6"/>
+<wire x1="109.22" y1="-17.78" x2="114.3" y2="-17.78" width="0.1524" layer="91"/>
+<label x="114.3" y="-17.78" size="1.27" layer="95" ratio="15" xref="yes"/>
+</segment>
 </net>
 <net name="PD.C" class="0">
@@
 </segment>
 </net>
-<net name="LED.CTRL" class="0">
+<net name="D29/LED.CTRL" class="0">
 <segment>
 <pinref part="U$4" gate="G$1" pin="A"/>
@@
 <wire x1="228.6" y1="33.02" x2="228.6" y2="40.64" width="0.1524" layer="91"/>
 <label x="228.6" y="40.64" size="1.27" layer="95" rot="R180" xref="yes"/>
+</segment>
+<segment>
+<pinref part="J1" gate="G$1" pin="4"/>
+<wire x1="109.22" y1="-22.86" x2="114.3" y2="-22.86" width="0.1524" layer="91"/>
+<label x="114.3" y="-22.86" size="1.27" layer="95" ratio="15" xref="yes"/>
 </segment>
 </net>
@@
 </segment>
 </net>
-<net name="PPG" class="0">
+<net name="A0/PPG" class="0">
 <segment>
 <wire x1="160.02" y1="30.48" x2="162.56" y2="30.48" width="0.1524" layer="91"/>
@@
 <label x="223.52" y="124.46" size="1.27" layer="95" rot="R180" xref="yes"/>
 <label x="223.52" y="104.14" size="1.27" layer="95" xref="yes"/>
+</segment>
+<segment>
+<pinref part="J1" gate="G$1" pin="5"/>
+<wire x1="109.22" y1="-20.32" x2="114.3" y2="-20.32" width="0.1524" layer="91"/>
+<label x="114.3" y="-20.32" size="1.27" layer="95" ratio="15" xref="yes"/>
 </segment>
 </net>
@@
 </segment>
 </net>
+<net name="N$6" class="0">
+<segment>
+<pinref part="J1" gate="G$1" pin="3"/>
+<wire x1="109.22" y1="-25.4" x2="114.3" y2="-25.4" width="0.1524" layer="91"/>
+</segment>
+</net>
+<net name="N$7" class="0">
+<segment>
+<pinref part="J1" gate="G$1" pin="2"/>
+<wire x1="109.22" y1="-27.94" x2="114.3" y2="-27.94" width="0.1524" layer="91"/>
+</segment>
+</net>
+<net name="N$11" class="0">
+<segment>
+<pinref part="J1" gate="G$1" pin="1"/>
+<wire x1="109.22" y1="-30.48" x2="114.3" y2="-30.48" width="0.1524" layer="91"/>
+</segment>
+</net>

Commit message: finished routing all boards
Parts:
- removed J1: (no value), LinnesLab-Connectors:CONN_07
- added C1: 100n, LinnesLab-Passives:CAPACITOR0603
- added C2: 1u, LinnesLab-Passives:CAPACITOR0603
- added J2: (no value), LinnesLab-Connectors:CONN_07-1.27MM
- added U3: PCF8523, LinnesLab-Clocks:PCF8523
- added XTAL2: 32.7680kHz, LinnesLab-Clocks:CRYSTALECS-.327-12.5-12-C-TR
Connections:
- removed net LED: Q1.C
- removed net N$11: J1.1
- removed net N$6: J1.3
- removed net N$7: J1.2
- new net N$1: U3.OSCO, XTAL2.1
- new net N$2: U3.OSCI, XTAL2.2
- new net VBATT: U3.VBAT
- net 3.3V: now also C2.1, J2.4, U3.VDD
- net A0/PPG: now also J2.7; no longer J1.5
- net A7/TIA: now also J2.6; no longer J1.6
- net D29/LED.CTRL: now also J2.5; no longer J1.4
- net GND: now also C1.1, C2.2, J2.3, U3.VSS
- net LED.C: now also Q1.C
- net SCL: now also J2.2, U3.SCL
- net SDA: now also J2.1, U3.SDA
- net VREF: now also C1.2
Other:
- note added: "Accelerometer"
- note added: "Back-up battery if desired"
- note added: "Castallated IMU Breakout"
- note added: "Connection to Digital Potentiometer for dynamic gain control"
- note added: "Connection to Optical Sensor Module"
- note added: "Connection to Upper Board"
- note added: "I2C Address = 0x68h"
- note added: "Real-Time Clock"
- note added: "VREF Generator and Bypass Capacitor"
- note added: "Winston PPG Circuit"
- moved on the sheet: C10, C11, C14, C15, C16, C17, C18, C19, C20, C21, C22, C24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
