File: Hardware/Top/Winston-TOP.sch (EAGLE design)
At the start: 52 parts, among them SW1 SWITCH.MOM, SW2 SWITCH.MOM, SW5 SWITCH.MOM, U2 NRF52832_MODULE_MDBT42, U4 PCF8523

Commit message: updated Hardware files
Parts:
- added C22: 100n, LinnesLab-Passives:CAPACITOR0603
- added C23, C24: 47p, LinnesLab-Passives:CAPACITOR0603
- added JP2: (no value), LinnesLab-Switches:JUMPER-SMT_2_NO_SILK
- added LED5: RED, LinnesLab-LED:LED0603
- added LED6: YELLOW, LinnesLab-LED:LED0603
- added R1, R2: 0, LinnesLab-Passives:RESISTOR0603
- added R17, R18: 27, LinnesLab-Passives:RESISTOR0603
- added R19, R20: 1k, LinnesLab-Passives:RESISTOR0603
- added U5: FT231XS, LinnesLab-DigitalIC:FT231XS
- R8, R9: value 10k -> 10K
Connections:
- removed net RXD: U2.P0.08
- removed net TXD: U2.P0.06
- new net !CTS: JP2.2, U5.!CTS
- new net FT3V3: U5.3V3OUT
- new net N$23: R17.2, U5.USBDM
- new net N$24: R18.2, U5.USBDP
- new net N$25: LED5.C, R19.2
- new net N$26: LED6.C, R20.2
- new net RXD.FT: R2.1, U5.RXD
- new net RXD.NRF: R1.2, U2.P0.08
- new net RXLED: R19.1, U5.CBUS1
- new net TXD.FT: R1.1, U5.TXD
- new net TXD.NRF: R2.2, U2.P0.06
- new net TXLED: R20.1, U5.CBUS2
- net 3.3V: now also C22.2, LED5.A, LED6.A, U5.!RESET, U5.VCCIO
- net DTR: now also U5.!DTR
- net GND: now also C22.1, C23.2, C24.1, JP2.1, U5.GND@16, U5.GND@6
- net SCL: now also R9.1; no longer R8.1
- net SDA: now also R8.1; no longer R9.1
- net USB+: now also C23.1, R18.1
- net USB-: now also C24.2, R17.1
- net V_USB: now also U5.VCC
Other:
- note added: "Added I2C pull-up resistor. All I2C pins share this same resistor"
- note added: "I don't remember if CTS needs to be grounded or left floating so here's a jumper to ground so it can be configued either way dynamically."
- note added: "Serial Programming Chip"
- note added: "TXD goes to RX on the other device RXD goes to TX on the other device"
- moved on the sheet: R8, R9

Commit message: updated top and bottom boards with everything from Take 002
Parts:
- added J3: (no value), LinnesLab-Connectors:CONN_061.27MM
Connections:
- removed net BATT: R13.1, R14.2
- removed net CD1: SD2.CARD_DETECT
- removed net CHRG.STAT: CHRG2.STAT, R12.1
- removed net CS.OLED: U3./CS
- removed net DC.OLED: U3.DC/I2C_SA0
- removed net RESET.OLED: U3./RES
- removed net SD.CS: SD2.CS
- removed net SW1: SW1.1, SW2.1, SW5.1
- new net A0/PPG: J3.5, U2.P0.02/AIN0
- new net A4/BATT: R13.1, R14.2, U2.P0.28/AIN4
- new net A7/TIA: J3.6, U2.P0.31/AIN7
- new net D11/SW1: SW1.1, U2.P0.11
- new net D15/SW2: SW2.1, U2.P0.15
- new net D16/SW3: SW5.1, U2.P0.16
- new net D27/CHRG.STATUS: CHRG2.STAT, R12.1, U2.P0.27
- new net D29/LED.CTRL: J3.4, U2.P0.29/AIN5
- new net D3/RESET.OLED: U2.P0.03/AIN1, U3./RES
- new net D30/CS.OLED: U2.P0.30/AIN6, U3./CS
- new net D4/DC.OLED: U2.P0.04/AIN2, U3.DC/I2C_SA0
- new net D5/CD1: SD2.CARD_DETECT, U2.P0.05/AIN3
- new net D7/SD.CS: SD2.CS, U2.P0.07
- new net N$22: J3.3
- new net N$27: J3.2
- new net N$28: J3.1
Other:
- note added: "Digital Charge Status Output"
- note added: "FDTI Serial to USB Converter"
- note added: "Serial programming chip converts USB protocol to serial protocol, which allows you to program the microcontroller via USB"
- note removed: "Serial Programming Chip"

Commit message: routed the top board
Parts:
- removed C14, C22: 100n, LinnesLab-Passives:CAPACITOR0603
- removed C15, C17: 2.2uF, LinnesLab-Passives:CAPACITOR0402
- removed C23, C24: 47p, LinnesLab-Passives:CAPACITOR0603
- removed CHRG2: MCP73831, LinnesLab-Power:MCP73831
- removed D4: (no value), LinnesLab-DiscreteSemi:SCHOTTKY-USC
- removed J3: (no value), LinnesLab-Connectors:CONN_061.27MM
- removed LDO2: MIC5504, LinnesLab-Power:MIC5504
- removed LED5: RED, LinnesLab-LED:LED0603
- removed LED6: YELLOW, LinnesLab-LED:LED0603
- removed R19: 1k, LinnesLab-Passives:RESISTOR0603
- removed R5: 10k, LinnesLab-Passives:RESISTOR0603
- removed R8, R9: 10K, LinnesLab-Passives:RESISTOR0603
- removed U5: FT231XS, LinnesLab-DigitalIC:FT231XS
- removed XTAL3: 32.7680kHz, LinnesLab-Clocks:CRYSTALECS-.327-12.5-12-C-TR
- added C3: 2.2uF, LinnesLab-Passives:CAPACITOR0402
- added D3: (no value), LinnesLab-DiscreteSemi:SCHOTTKY-USC
- added J1: (no value), LinnesLab-Connectors:CONN_07-1.27MM
- added LED1: RED, LinnesLab-LED:LED0603
- added LED2: BLUE, LinnesLab-LED:LED0603
- added R10: 100k, LinnesLab-Passives:RESISTOR0603
- C10: value 300p -> (none)
- C12: value 10u -> 300p; device LinnesLab-Passives:CAPACITOR0805 -> LinnesLab-Passives:CAPACITOR0603
- C18, C19: value 2.2uF -> 47p; device LinnesLab-Passives:CAPACITOR0402 -> LinnesLab-Passives:CAPACITOR0603
- C2, C5, C6: value 1u -> 2.2uF; device LinnesLab-Passives:CAPACITOR0603 -> LinnesLab-Passives:CAPACITOR0402
- C20, C21: value 4.7u -> 100n
- C8: value (none) -> 10u; device LinnesLab-Passives:CAPACITOR0603 -> LinnesLab-Passives:CAPACITOR0805
- LED4: value BLUE -> YELLOW
- R1: value 0 -> 10k
- R11: value (none) -> 100k
- R12, R13: value 100k -> 27
- R14: value 100k -> 10k
- R15: value 100k -> 1k
- R17, R18: value 27 -> 0
- R2: value 0 -> 390k
- R3, R4: value 1k -> 10K
- R6: value 10k -> 1k
- R7: value 390k -> 1k
- SW3: value (none) -> SWITCH.MOM; device LinnesLab-Switches:SPST-PTS830GG140-COPY.1-3 -> LinnesLab-Switches:SWITCH.MOM
- SW5: value SWITCH.MOM -> (none); device LinnesLab-Switches:SWITCH.MOM -> LinnesLab-Switches:SPST-PTS830GG140-COPY.1-3
- U4: value PCF8523 -> FT231XS; device LinnesLab-Clocks:PCF8523 -> LinnesLab-DigitalIC:FT231XS; DIGIKEY 568-5306-1-ND -> (none); I2C_ADDRESS 0x68h -> (none); MFN PCF8523T/1,118 -> (none); MFN_MANUFACTURER NXP USA Inc. -> (none)
- renumbered C13 to C4, C16 to C1, CORTEX1 to DEBUG1, D5 to D2, JP2 to JP1, L2 to L1, R20 to R16, SD2 to SD1, U3 to U1, USB2 to USB1, XTAL2 to XTAL1
Connections:
- removed net N$17: CHRG2.PROG, R11.2
- removed net N$19: U4.OSCO, XTAL3.1
- removed net N$20: U4.OSCI, XTAL3.2
- removed net N$22: J3.3
- removed net N$27: J3.2
- removed net N$28: J3.1
- removed net VBATT: U4.VBAT
- net !CTS: now also U4.!CTS; no longer U5.!CTS
- net 3.3V: now also C20.2, C5.2, C6.2, C8.2, D3.C, J1.4, LED3.A, LED4.A, R14.2, R3.2, R4.2, U4.!RESET, U4.VCCIO; no longer C12.2, C17.2, C19.2, C2.1, C22.2, C6.1, D1.C, LDO2.OUT, LED5.A, LED6.A, R15.2, R5.2, R8.2, R9.2, U4.VDD, U5.!RESET, U5.VCCIO
- net A0/PPG: now also J1.7; no longer J3.5
- net A4/BATT: now also R10.1, R11.2; no longer R13.1, R14.2
- net A7/TIA: now also J1.6; no longer J3.6
- net D16/SW3: now also SW3.1; no longer SW5.1
- net D27/CHRG.STATUS: no longer CHRG2.STAT, R12.1
- net D29/LED.CTRL: now also J1.5; no longer J3.4
- net DFU: now also SW4.B; no longer SW3.B
- net DTR: now also C21.1, U4.!DTR; no longer C14.1, U5.!DTR
- net FT3V3: now also U4.3V3OUT; no longer U5.3V3OUT
- net GND: now also C12.2, C19.2, C20.1, C3.1, C6.1, C9.1, J1.3, LED1.C, LED2.C, R1.1, R2.2, SW3.3, SW3.4, SW4.A, SW5.B, U4.GND@16, U4.GND@6; no longer C12.1, C17.1, C19.1, C2.2, C20.2, C21.1, C22.1, C23.2, C24.1, C6.2, C9.2, CHRG2.VSS, LDO2.GND, LED3.C, LED4.C, R14.1, R15.1, R6.1, R7.2, SW3.A, SW4.B, SW5.3, SW5.4, U4.VSS, U5.GND@16, U5.GND@6
- net LED1: now also R6.2; no longer R3.2
- net LED2: now also R7.2; no longer R4.2
- net N$1: now also R1.2; no longer R6.2
- net N$10: now also LED2.A, R7.1; no longer LED4.A, R4.1
- net N$15: now also C3.2; no longer C18.2
- net N$2: now also R2.1; no longer R7.1
- net N$23: now also R12.2, U4.USBDM; no longer R17.2, U5.USBDM
- net N$24: now also R13.2, U4.USBDP; no longer R18.2, U5.USBDP
- net N$25: now also LED3.C, R15.2; no longer LED5.C, R19.2
- net N$26: now also LED4.C; no longer LED6.C
- net N$4: now also C9.2; no longer C8.2
- net N$6: now also C10.1; no longer C9.1
- net N$7: now also C2.2; no longer C15.2
- net N$8: now also C2.1; no longer C15.1
- net N$9: now also LED1.A, R6.1; no longer LED3.A, R3.1
- net P0.10/NFC2: now also C12.1; no longer C10.1
- net RESET: now also C21.2, D3.A, R14.1, SW5.A; no longer C14.2, D1.A, R5.1, SW4.A
- net RXD.FT: now also R18.1, U4.RXD; no longer R2.1, U5.RXD
- net RXD.NRF: now also R17.2; no longer R1.2
- net RXLED: now also R15.1, U4.CBUS1; no longer R19.1, U5.CBUS1
- net SCL: now also J1.2, R4.1; no longer R9.1, U4.SCL
- net SDA: now also J1.1, R3.1; no longer R8.1, U4.SDA
- net TXD.FT: now also R17.1, U4.TXD; no longer R1.1, U5.TXD
- net TXD.NRF: now also R18.2; no longer R2.2
- net TXLED: now also U4.CBUS2; no longer U5.CBUS2
- net USB+: now also C19.1, R13.1; no longer C23.1, R18.1
- net USB-: now also C18.2, R12.1; no longer C24.2, R17.1
- net VIN: now also D1.C; no longer C21.2, C5.2, CHRG2.VIN, D4.C, LDO2.EN, LDO2.IN, R12.2
- net VLIPO: now also D1.A, R10.2; no longer C20.1, CHRG2.VBAT, D4.A, R13.2
- net V_USB: now also U4.VCC; no longer U5.VCC
Other:
- note added: "Connection To Bottom Board"
- note removed: "Back-up battery if desired"
- note removed: "Digital Charge Status Output"
- note removed: "I2C Address = 0x68h"
- note removed: "Real-Time Clock"
- moved on the sheet: C10, C12, C18, C19, C2, C20, C21, C5, C6, C8, C9, D1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

Commit message: finished routing all boards
Parts:
- removed C21: 100n, LinnesLab-Passives:CAPACITOR0603
- removed R18: 0, LinnesLab-Passives:RESISTOR0603
- added C13, C16: 4.7u, LinnesLab-Passives:CAPACITOR0603
- added C14, C15: 1u, LinnesLab-Passives:CAPACITOR0603
- added C17: 47p, LinnesLab-Passives:CAPACITOR0603
- added CHRG1: MCP73831, LinnesLab-Power:MCP73831
- added LDO1: MIC5504, LinnesLab-Power:MIC5504
- added R5, R9: 100k, LinnesLab-Passives:RESISTOR0603
- added R8: (no value), LinnesLab-Passives:RESISTOR0603
- C19: value 47p -> 100n
- R11: value 100k -> 27
- R13: value 27 -> 10k
- R14: value 10k -> 1k
- R16: value 1k -> 0
- renumbered U4 to U3
Connections:
- new net N$16: CHRG1.PROG, R8.2
- net 3.3V: now also C15.1, C19.2, LDO1.OUT, R13.2; no longer C20.2, R14.2
- net A4/BATT: now also R10.2, R9.1; no longer R10.1, R11.2
- net D27/CHRG.STATUS: now also CHRG1.STAT, R5.1
- net DTR: now also C20.1; no longer C21.1
- net GND: now also C13.1, C14.1, C15.2, C16.2, C17.1, C18.2, C19.1, CHRG1.VSS, LDO1.GND, R10.1, R8.1; no longer C18.1, C19.2, C20.1, R11.1
- net N$23: now also R11.2; no longer R12.2
- net N$24: now also R12.2; no longer R13.2
- net N$25: now also R14.2; no longer R15.2
- net N$26: now also R15.2; no longer R16.2
- net RESET: now also C20.2, R13.1; no longer C21.2, R14.1
- net RXD.FT: now also R17.1; no longer R18.1
- net RXD.NRF: now also R16.2; no longer R17.2
- net RXLED: now also R14.1; no longer R15.1
- net TXD.FT: now also R16.1; no longer R17.1
- net TXD.NRF: now also R17.2; no longer R18.2
- net TXLED: now also R15.1; no longer R16.1
- net USB+: now also C18.1, R12.1; no longer C19.1, R13.1
- net USB-: now also C17.2, R11.1; no longer C18.2, R12.1
- net VIN: now also C13.2, C14.2, CHRG1.VIN, LDO1.EN, LDO1.IN, R5.2
- net VLIPO: now also C16.1, CHRG1.VBAT, R9.2; no longer R10.2
Other:
- note added: "Digital Charge Status Output"
- moved on the sheet: C18, C19, C20, R10, R11, R12, R13, R14, R15, R16, R17

Commit message: continued routing top board
Parts:
- removed C11, C12: 300p, LinnesLab-Passives:CAPACITOR0603
Connections:
- net GND: no longer C11.2, C12.2
- net P0.09/NFC1: no longer C11.1
- net P0.10/NFC2: no longer C12.1
Changed lines of the file:
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@@
 <part name="GND15" library="LinnesLab-Symbols" deviceset="GND" device=""/>
 <part name="GND16" library="LinnesLab-Symbols" deviceset="GND" device=""/>
-<part name="GND17" library="LinnesLab-Symbols" deviceset="GND" device=""/>
-<part name="GND18" library="LinnesLab-Symbols" deviceset="GND" device=""/>
 <part name="GND19" library="LinnesLab-Symbols" deviceset="GND" device=""/>
 <part name="GND20" library="LinnesLab-Symbols" deviceset="GND" device=""/>
@@
 <part name="C9" library="LinnesLab-Passives" deviceset="CAPACITOR" device="0603" package3d_urn="urn:adsk.eagle:package:15661989/2"/>
 <part name="C10" library="LinnesLab-Passives" deviceset="CAPACITOR" device="0603" package3d_urn="urn:adsk.eagle:package:15661989/2"/>
-<part name="C12" library="LinnesLab-Passives" deviceset="CAPACITOR" device="0603" package3d_urn="urn:adsk.eagle:package:15661989/2" value="300p"/>
-<part name="C11" library="LinnesLab-Passives" deviceset="CAPACITOR" device="0603" package3d_urn="urn:adsk.eagle:package:15661989/2" value="300p"/>
 <part name="C8" library="LinnesLab-Passives" deviceset="CAPACITOR" device="0805" package3d_urn="urn:adsk.eagle:package:15662010/2" value="10u"/>
 <part name="L1" library="LinnesLab-Passives" deviceset="INDUCTOR" device="0603" override_package3d_urn="urn:adsk.eagle:package:18592195/2" override_package_urn="urn:adsk.eagle:footprint:18592196/1" value="10u"/>
@@
 <attribute name="VALUE" x="154.94" y="98.806" size="1.778" layer="96" align="top-center"/>
 </instance>
-<instance part="GND17" gate="G$1" x="157.48" y="68.58" smashed="yes">
-<attribute name="VALUE" x="157.48" y="68.326" size="1.778" layer="96" align="top-center"/>
-</instance>
-<instance part="GND18" gate="G$1" x="144.78" y="68.58" smashed="yes">
-<attribute name="VALUE" x="144.78" y="68.326" size="1.778" layer="96" align="top-center"/>
-</instance>
 <instance part="GND19" gate="G$1" x="134.62" y="68.58" smashed="yes">
 <attribute name="VALUE" x="134.62" y="68.326" size="1.778" layer="96" align="top-center"/>
@@
 <attribute name="NAME" x="136.144" y="79.121" size="1.778" layer="95"/>
 <attribute name="VALUE" x="136.144" y="74.041" size="1.778" layer="96"/>
-</instance>
-<instance part="C12" gate="G$1" x="157.48" y="76.2" smashed="yes">
-<attribute name="NAME" x="159.004" y="79.121" size="1.778" layer="95"/>
-<attribute name="VALUE" x="159.004" y="74.041" size="1.778" layer="96"/>
-</instance>
-<instance part="C11" gate="G$1" x="144.78" y="76.2" smashed="yes">
-<attribute name="NAME" x="146.304" y="79.121" size="1.778" layer="95"/>
-<attribute name="VALUE" x="146.304" y="74.041" size="1.778" layer="96"/>
 </instance>
 <instance part="C8" gate="G$1" x="114.3" y="111.76" smashed="yes" rot="R180">
@@
 <pinref part="GND20" gate="G$1" pin="GND"/>
 <pinref part="C9" gate="G$1" pin="1"/>
-</segment>
-<segment>
-<pinref part="C11" gate="G$1" pin="2"/>
-<pinref part="GND18" gate="G$1" pin="GND"/>
-<wire x1="144.78" y1="71.12" x2="144.78" y2="73.66" width="0.1524" layer="91"/>
-</segment>
-<segment>
-<pinref part="C12" gate="G$1" pin="2"/>
-<pinref part="GND17" gate="G$1" pin="GND"/>
-<wire x1="157.48" y1="71.12" x2="157.48" y2="73.66" width="0.1524" layer="91"/>
 </segment>
 <segment>
@@
 <segment>
 <wire x1="149.86" y1="104.14" x2="149.86" y2="83.82" width="0.1524" layer="91"/>
-<wire x1="144.78" y1="83.82" x2="149.86" y2="83.82" width="0.1524" layer="91"/>
-<wire x1="144.78" y1="83.82" x2="144.78" y2="81.28" width="0.1524" layer="91"/>
-<pinref part="C11" gate="G$1" pin="1"/>
 <pinref part="U2" gate="G$1" pin="P0.09"/>
 <label x="149.86" y="86.36" size="1.27" layer="95" rot="R180" xref="yes"/>
@@
 <segment>
 <wire x1="152.4" y1="104.14" x2="152.4" y2="83.82" width="0.1524" layer="91"/>
-<wire x1="152.4" y1="83.82" x2="157.48" y2="83.82" width="0.1524" layer="91"/>
-<wire x1="157.48" y1="83.82" x2="157.48" y2="81.28" width="0.1524" layer="91"/>
-<pinref part="C12" gate="G$1" pin="1"/>
 <pinref part="U2" gate="G$1" pin="P0.10"/>
 <label x="152.4" y="86.36" size="1.27" layer="95" xref="yes"/>
