File: Hardware/Top/Winston-TOP.brd (EAGLE design)
At the start: 38 x 38 mm, 60 parts, among them SW1 SWITCH.MOM, SW2 SWITCH.MOM, SW3 SWITCH.MOM, U2 NRF52832_MODULE_MDBT42, U3 FT231XS

Commit message: Completed Routing Top Board
Parts:
- moved R1 2.80 mm to (14.2, 21.0)
- moved C3 2.00 mm to (25.9, 13.5)
- moved R6 1.48 mm to (33.4, 20.2)
- moved LED3 1.38 mm to (18.1, 7.20)
- moved LED1 1.25 mm to (33.4, 17.1)
- moved R2 1.02 mm to (24.4, 14.8)
- moved C1 0.98 mm to (29.0, 15.6), turned to 180 degrees
- moved R7 0.92 mm to (34.9, 21.1)
- moved C7 0.90 mm to (20.5, 29.0)
- moved XTAL1 0.64 mm to (20.3, 22.0)
- moved C6 0.63 mm to (12.6, 22.7)
- moved L1 0.62 mm to (20.5, 25.7)
- moved LED2 0.59 mm to (34.9, 18.1)
- moved R8 0.50 mm to (3.55, 18.6)
- moved C9 0.45 mm to (17.4, 23.1)
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Routing:
- net RESET: track 11.2 -> 30.5 mm
- net GND: track 65.5 -> 73.2 mm, vias 41 -> 42
- net SWO: track 5.05 -> 11.6 mm, vias 0 -> 1
- net N$1: track 5.99 -> 3.21 mm
- net SWDIO: track 6.68 -> 4.60 mm
- net LED2: track 9.54 -> 11.6 mm
- net SWCLK: track 7.77 -> 9.50 mm, vias 0 -> 1
- net N$15: track 2.37 -> 4.06 mm
- net 3.3V: track 0.00 -> 1.48 mm, vias 0 -> 1
- net D5/CD1: track 30.6 -> 29.4 mm, vias 1 -> 3
- net N$2: track 2.90 -> 4.07 mm
- net LED1: track 8.86 -> 9.84 mm
- net DTR: track 24.3 -> 25.1 mm
- net N$12: track 4.85 -> 4.11 mm
- net A4/BATT: track 28.0 -> 27.3 mm
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